Commit message: updates

File: robot_description/include/_d435i.urdf.xacro (robot description, xacro)
@@ -7,5 +7,5 @@
 -->
 <robot name="sensor_d435i" xmlns:xacro="http://ros.org/wiki/xacro">
-  <xacro:include filename="$(find raptor_description)/urdf/include/_d435.urdf.xacro"/>
+  <xacro:include filename="$(find raptor_v2)/robot_description/include/_d435.urdf.xacro"/>
   <xacro:include filename="$(find realsense2_description)/urdf/_d435i_imu_modules.urdf.xacro"/>
   <xacro:macro name="sensor_d435i" params="parent name:=camera use_nominal_extrinsics:=false">

File: robot_description/include/gazebo.xacro (robot description, xacro)
@@ -82,24 +82,3 @@
   <slip2>1.0</slip2>
 </gazebo>
-<gazebo reference="bucket">
-  <material>Gazebo/Blue</material>
-</gazebo>
-<gazebo reference="head">
-  <material>Gazebo/Yellow</material>
-</gazebo>
-<gazebo reference="pvc_horizontal">
-  <material>Gazebo/Yellow</material>
-</gazebo>
-<gazebo reference="pvc_up_left">
-  <material>Gazebo/Yellow</material>
-</gazebo>
-<gazebo reference="pvc_up_right">
-  <material>Gazebo/Yellow</material>
-</gazebo>
-<gazebo reference="pvc_45_left">
-  <material>Gazebo/Yellow</material>
-</gazebo>
-<gazebo reference="pvc_45_right">
-  <material>Gazebo/Yellow</material>
-</gazebo>
 </robot>

File: robot_description/raptor.urdf.xacro (robot description, xacro)
@@ -1,7 +1,7 @@
 <?xml version="1.0"?>
 	<robot name="raptor" xmlns:xacro="http://www.ros.org/wiki/xacro">
-	<xacro:include filename="$(find raptor_description)/urdf/include/material.xacro"/>
-	<xacro:include filename="$(find raptor_description)/urdf/include/gazebo.xacro"/>
-	<xacro:include filename="$(find raptor_description)/urdf/include/_d435i.urdf.xacro"/>
+	<xacro:include filename="$(find raptor_v2)/robot_description/include/material.xacro"/>
+	<xacro:include filename="$(find raptor_v2)/robot_description/include/gazebo.xacro"/>
+	<xacro:include filename="$(find raptor_v2)/robot_description/include/_d435i.urdf.xacro"/>
   		<link name="base_link">
 		</link>
